File: PCB/ATF150x_uDEV.kicad_sch (KiCad schematic)
At the start: 14 parts, among them J1 Altera JTAG-A+VPP, J2 1x20x2.54mm, J3 1x20x2.54mm, U1 ATF150x-xAx44

Commit message: mpns & bom
Parts:
- C1, C2, C3, C4: MPN (none) -> CL21B105KOFNNWE
- J1: MPN (none) -> SBH11-PBPC-D05-ST-BK
- J2, J3: MPN (none) -> PRPC020SAAN-RC
- JP1: symbol Jumper:Jumper_2_Bridged -> 000_LOCAL:Jumper_2_Bridged; MPN (none) -> PRPC002SBBN-M71RC
- LED1, LED2: MPN 150060GS75000 -> LG_R971-KN-1-0-20-R18; Mfg Wurth -> (none)
- R1, R2: MPN (none) -> RMCF0805FT10K0
- U1: MPN (none) -> ATF1504ASL-25AU44
Other:
- note added: "Additional BOM part, jumper for JP1, typical: Sullins SPC02SYAN"
